Commit message: fixes in urdf

File: src/drone_description/description/core.xacro (robot description, xacro)
@@ -2,26 +2,4 @@
 <robot xmlns:xacro="http://ros.org">
     <xacro:include filename="inertial.xacro" />
-    <link name="world"></link>
-    <joint name="world_joint" type="fixed">
-        <parent link="world" />
-        <child link="base_link" />
-        <origin xyz="0 0 0.1" rpy="0 0 0" />
-    </joint>
-    <link name="base_link">
-        <visual>
-            <geometry>
-                <box size="0.3 0.3 0.05" />
-            </geometry>
-        </visual>
-        <collision>
-            <geometry>
-                <box size="0.3 0.3 0.05" />
-            </geometry>
-        </collision>
-        <xacro:inertial_box mass="1.0" x="0.3" y="0.3" z="0.05">
-            <origin xyz="0 0 0" rpy="0 0 0" />
-        </xacro:inertial_box>
-    </link>
-    <!-- Macro για έλικες (0-3) -->
     <xacro:macro name="rotor" params="suffix x y">
         <joint name="rotor_${suffix}_joint" type="continuous">
@@ -42,7 +20,3 @@
         </link>
     </xacro:macro>
-    <xacro:rotor suffix="0" x="0.15" y="0.15" />
-    <xacro:rotor suffix="1" x="-0.15" y="-0.15" />
-    <xacro:rotor suffix="2" x="0.15" y="-0.15" />
-    <xacro:rotor suffix="3" x="-0.15" y="0.15" />
 </robot>

File: src/drone_description/description/drone.urdf.xacro (robot description, xacro)
@@ -5,3 +5,35 @@
     <xacro:include filename="sensors.xacro" />
     <xacro:include filename="ardupilot_plugin.xacro" />
+    <link name="base_footprint"/>
+    <joint name="base_joint" type="fixed">
+        <parent link="base_footprint"/>
+        <child link="base_link"/>
+        <origin xyz="0 0 0" rpy="0 0 0"/>
+    </joint>
+    <link name="base_link">
+        <visual>
+            <geometry>
+                <box size="0.3 0.3 0.05" />
+            </geometry>
+        </visual>
+        <collision>
+            <geometry>
+                <box size="0.3 0.3 0.05" />
+            </geometry>
+        </collision>
+        <xacro:inertial_box mass="1.0" x="0.3" y="0.3" z="0.05">
+            <origin xyz="0 0 0" rpy="0 0 0" />
+        </xacro:inertial_box>
+    </link>
+    <xacro:rotor suffix="0" x="0.15" y="0.15" />
+    <xacro:rotor suffix="1" x="-0.15" y="-0.15" />
+    <xacro:rotor suffix="2" x="0.15" y="-0.15" />
+    <xacro:rotor suffix="3" x="-0.15" y="0.15" />
+    <!-- Το frame της κάμερας στην θέση που ορίζει το YAML (0.7, 0, 1.15) -->
+    <link name="camera_link"/>
+    <joint name="camera_joint" type="fixed">
+    <parent link="base_link"/>
+    <child link="camera_link"/>
+    <origin xyz="0.7 0.0 1.150" rpy="0 0 0"/>
+    </joint>
 </robot>
