Commit message: first version working point cloud

File: src/drone_description/description/sensors.xacro (robot description, xacro)
@@ -23,11 +23,12 @@
         </collision>
     </link>
+    <!-- RGB camera for color image -->
     <gazebo reference="camera_link">
-        <sensor name="camera" type="camera">
+        <sensor name="rgb_camera" type="camera">
             <always_on>true</always_on>
             <visualize>true</visualize>
             <update_rate>30</update_rate>
             <topic>camera/image_raw</topic>
-            <camera name="intel_realsense_r200">
+            <camera name="intel_realsense_rgb">
                 <optical_frame_id>camera_rgb_optical_frame</optical_frame_id>
                 <camera_info_topic>camera/camera_info</camera_info_topic>
@@ -46,4 +47,42 @@
         </sensor>
     </gazebo>
+    <link name="camera_rgb_optical_frame" />
+    <joint name="camera_rgb_optical_frame_joint" type="fixed">
+        <parent link="camera_link" />
+        <child link="camera_rgb_optical_frame" />
+        <origin xyz="0 0 0" rpy="-1.57079632679 0 -1.57079632679" />
+    </joint>
+    <!-- Depth camera implemented as a Gazebo Sim depth_camera sensor (publishes depth image;
+    Sensors
+    system will provide pointcloud) -->
+    <gazebo reference="camera_link">
+        <sensor name="depth_camera" type="depth_camera">
+            <always_on>true</always_on>
+            <visualize>true</visualize>
+            <update_rate>30</update_rate>
+            <topic>camera/depth/image_raw</topic>
+            <camera name="intel_realsense_depth">
+                <optical_frame_id>camera_depth_optical_frame</optical_frame_id>
+                <camera_info_topic>camera/depth/camera_info</camera_info_topic>
+                <horizontal_fov>1.05</horizontal_fov>
+                <pose>0 0 0 0 0 0</pose>
+                <image>
+                    <width>640</width>
+                    <height>480</height>
+                    <format>R_FLOAT32</format>
+                </image>
+                <clip>
+                    <near>0.1</near>
+                    <far>10.0</far>
+                </clip>
+            </camera>
+        </sensor>
+    </gazebo>
+    <link name="camera_depth_optical_frame" />
+    <joint name="camera_depth_optical_frame_joint" type="fixed">
+        <parent link="camera_link" />
+        <child link="camera_depth_optical_frame" />
+        <origin xyz="0 0 0" rpy="-1.57079632679 0 -1.57079632679" />
+    </joint>
     <joint name="camera_joint" type="fixed">
         <parent link="base_link" />
@@ -79,5 +118,4 @@
             <visualize>true</visualize>
             <topic>imu</topic>
-            <plugin name="gz::sim::systems::Imu" filename="gz-sim-imu-system" />
         </sensor>
     </gazebo>
