Commit message: imu added and adjustments

File: src/drone_description/description/drone.urdf.xacro (robot description, xacro)
@@ -5,9 +5,9 @@
     <xacro:include filename="sensors.xacro" />
     <xacro:include filename="ardupilot_plugin.xacro" />
-    <link name="base_footprint"/>
+    <link name="base_footprint" />
     <joint name="base_joint" type="fixed">
-        <parent link="base_footprint"/>
-        <child link="base_link"/>
-        <origin xyz="0 0 0" rpy="0 0 0"/>
+        <parent link="base_footprint" />
+        <child link="base_link" />
+        <origin xyz="0 0 0" rpy="0 0 0" />
     </joint>
     <link name="base_link">
@@ -30,10 +30,3 @@
     <xacro:rotor suffix="2" x="0.15" y="-0.15" />
     <xacro:rotor suffix="3" x="-0.15" y="0.15" />
-    <!-- Το frame της κάμερας στην θέση που ορίζει το YAML (0.7, 0, 1.15) -->
-    <link name="camera_link"/>
-    <joint name="camera_joint" type="fixed">
-    <parent link="base_link"/>
-    <child link="camera_link"/>
-    <origin xyz="0.7 0.0 1.150" rpy="0 0 0"/>
-    </joint>
 </robot>

File: src/drone_description/description/sensors.xacro (robot description, xacro)
@@ -1,4 +1,13 @@
 <?xml version="1.0"?>
 <robot xmlns:xacro="http://www.ros.org/wiki/xacro">
+    <!-- ===================== -->
+    <!-- IMU SENSOR (gz-sim)   -->
+    <!-- ===================== -->
+    <link name="camera_link" />
+    <joint name="camera_joint" type="fixed">
+        <parent link="base_link" />
+        <child link="camera_link" />
+        <origin xyz="0.7 0.0 1.150" rpy="0 0 0" />
+    </joint>
     <!-- ===================== -->
     <!-- IMU SENSOR (gz-sim)   -->

Commit message: working simple image and topics

File: src/drone_description/description/drone.urdf.xacro (robot description, xacro)
@@ -33,6 +33,13 @@
         <plugin filename="gz-sim-joint-state-publisher-system"
             name="gz::sim::systems::JointStatePublisher">
-            <!-- Optional: topic name defaults to /joint_states if omitted -->
             <topic>/drone/joint_states</topic>
+        </plugin>
+        <!-- <plugin
+            filename="gz-sim-physics-system"
+            name="gz::sim::systems::Physics">
+        </plugin> -->
+        <plugin
+            filename="gz-sim-scene-broadcaster-system"
+            name="gz::sim::systems::SceneBroadcaster">
         </plugin>
     </gazebo>

File: src/drone_description/description/sensors.xacro (robot description, xacro)
@@ -2,11 +2,52 @@
 <robot xmlns:xacro="http://www.ros.org/wiki/xacro">
     <!-- ===================== -->
-    <!-- IMU SENSOR (gz-sim)   -->
+    <!-- CAMERA -->
     <!-- ===================== -->
-    <link name="camera_link" />
+    <link name="camera_link">
+        <inertial>
+            <mass value="0.05" />
+            <inertia ixx="0.0001" ixy="0.0" ixz="0.0" iyy="0.0001" iyz="0.0" izz="0.0001" />
+        </inertial>
+        <visual>
+            <geometry>
+                <box size="0.02 0.08 0.02" />
+            </geometry>
+            <material name="red">
+                <color rgba="1 0 0 1" />
+            </material>
+        </visual>
+        <collision>
+            <geometry>
+                <box size="0.02 0.08 0.02" />
+            </geometry>
+        </collision>
+    </link>
+    <gazebo reference="camera_link">
+        <sensor name="camera" type="camera">
+            <always_on>true</always_on>
+            <visualize>true</visualize>
+            <update_rate>30</update_rate>
+            <topic>camera/image_raw</topic>
+            <camera name="intel_realsense_r200">
+                <optical_frame_id>camera_rgb_optical_frame</optical_frame_id>
+                <camera_info_topic>camera/camera_info</camera_info_topic>
+                <horizontal_fov>1.05</horizontal_fov>
+                <pose>0 0 0 0 0 0</pose>
+                <image>
+                    <width>640</width>
+                    <height>480</height>
+                    <format>R8G8B8</format>
+                </image>
+                <clip>
+                    <near>0.1</near>
+                    <far>10.0</far>
+                </clip>
+            </camera>
+        </sensor>
+    </gazebo>
     <joint name="camera_joint" type="fixed">
         <parent link="base_link" />
         <child link="camera_link" />
-        <origin xyz="0.7 0.0 1.150" rpy="0 0 0" />
+        <origin xyz="0.2 0 0.0" rpy="0 0 0" />
     </joint>
     <!-- ===================== -->
@@ -14,25 +55,44 @@
     <!-- ===================== -->
     <link name="imu_link">
+        <inertial>
+            <mass value="0.05" />
+            <inertia ixx="0.0001" ixy="0.0" ixz="0.0" iyy="0.0001" iyz="0.0" izz="0.0001" />
+        </inertial>
+        <visual>
+            <geometry>
+                <box size="0.02 0.02 0.02" />
+            </geometry>
+            <material name="blue">
+                <color rgba="0 0 1 1" />
+            </material>
+        </visual>
+        <collision>
+            <geometry>
+                <box size="0.02 0.02 0.02" />
+            </geometry>
+        </collision>
+    </link>
+    <gazebo reference="imu_link">
         <sensor name="imu_sensor" type="imu">
-            <always_on>true</always_on>
-            <update_rate>100</update_rate>
-            <visualize>false</visualize>
-            <!-- Gazebo Sim system plugin -->
-            <plugin name="imu_system" filename="gz-sim-imu-system" />
+            <always_on>1</always_on>
+            <update_rate>1</update_rate>
+            <visualize>true</visualize>
+            <topic>imu</topic>
+            <plugin name="gz::sim::systems::Imu" filename="gz-sim-imu-system" />
         </sensor>
-    </link>
-    <joint name="imu_joint" type="fixed">
+    </gazebo>
+    <joint
+        name="imu_joint" type="fixed">
         <parent link="base_link" />
         <child link="imu_link" />
     </joint>
-    <!-- ===================== -->
+    <!-- =====================  -->
     <!-- GPS SENSOR (gz-sim)   -->
     <!-- ===================== -->
-    <link name="gps_link">
+    <!-- <link name="gps_link">
         <sensor name="navsat_sensor" type="navsat">
             <always_on>true</always_on>
             <update_rate>10</update_rate>
             <visualize>false</visualize>
-            <!-- Gazebo Sim system plugin -->
             <plugin name="navsat_system" filename="gz-sim-navsat-system" />
         </sensor>
@@ -41,4 +101,11 @@
         <parent link="base_link" />
         <child link="gps_link" />
-    </joint>
+    </joint> -->
+    <gazebo>
+        <plugin
+            filename="gz-sim-sensors-system"
+            name="gz::sim::systems::Sensors">
+            <render_engine>ogre2</render_engine>
+        </plugin>
+    </gazebo>
 </robot>

Commit message: rgbd

File: src/drone_description/description/drone.urdf.xacro (robot description, xacro)
@@ -1,4 +1,5 @@
 <?xml version="1.0"?>
 <robot xmlns:xacro="http://www.ros.org/wiki/xacro" name="drone">
+    <xacro:property name="robot_namespace" value="drone" />
     <xacro:include filename="components/shapes.xacro" />
     <xacro:include filename="components/rotor.xacro" />
@@ -33,10 +34,6 @@
         <plugin filename="gz-sim-joint-state-publisher-system"
             name="gz::sim::systems::JointStatePublisher">
-            <topic>/drone/joint_states</topic>
+            <topic>/${robot_namespace}/joint_states</topic>
         </plugin>
-        <!-- <plugin
-            filename="gz-sim-physics-system"
-            name="gz::sim::systems::Physics">
-        </plugin> -->
         <plugin
             filename="gz-sim-scene-broadcaster-system"

File: src/drone_description/description/sensors.xacro (robot description, xacro)
@@ -23,16 +23,19 @@
         </collision>
     </link>
-    <!-- RGB camera for color image -->
+    <joint name="camera_joint" type="fixed">
+        <parent link="base_link" />
+        <child link="camera_link" />
+        <origin xyz="0.2 0 0.0" rpy="0 0 0" />
+    </joint>
     <gazebo reference="camera_link">
-        <sensor name="rgb_camera" type="camera">
-            <always_on>true</always_on>
+        <!-- Αλλαγή του type σε rgbd_camera -->
+        <sensor name="drone_rgbd_camera" type="rgbd_camera">
+            <always_on>1</always_on>
+            <update_rate>30</update_rate>
             <visualize>true</visualize>
-            <update_rate>30</update_rate>
-            <topic>camera/image_raw</topic>
-            <camera name="intel_realsense_rgb">
-                <optical_frame_id>camera_rgb_optical_frame</optical_frame_id>
-                <camera_info_topic>camera/camera_info</camera_info_topic>
-                <horizontal_fov>1.05</horizontal_fov>
-                <pose>0 0 0 0 0 0</pose>
+            <topic>/${robot_namespace}/camera/rgbd</topic>
+            <camera>
+                <optical_frame_id>camera_rgbd_optical_frame</optical_frame_id>
+                <horizontal_fov>1.047</horizontal_fov>
                 <image>
                     <width>640</width>
@@ -41,5 +44,5 @@
                 </image>
                 <clip>
-                    <near>0.1</near>
+                    <near>0.05</near>
                     <far>10.0</far>
                 </clip>
@@ -47,46 +50,9 @@
         </sensor>
     </gazebo>
-    <link name="camera_rgb_optical_frame" />
-    <joint name="camera_rgb_optical_frame_joint" type="fixed">
+    <link name="camera_rgbd_optical_frame" />
+    <joint name="camera_rgbd_optical_frame_joint" type="fixed">
         <parent link="camera_link" />
-        <child link="camera_rgb_optical_frame" />
-        <origin xyz="0 0 0" rpy="-1.57079632679 0 -1.57079632679" />
-    </joint>
-    <!-- Depth camera implemented as a Gazebo Sim depth_camera sensor (publishes depth image;
-    Sensors
-    system will provide pointcloud) -->
-    <gazebo reference="camera_link">
-        <sensor name="depth_camera" type="depth_camera">
-            <always_on>true</always_on>
-            <visualize>true</visualize>
-            <update_rate>30</update_rate>
-            <topic>camera/depth/image_raw</topic>
-            <camera name="intel_realsense_depth">
-                <optical_frame_id>camera_depth_optical_frame</optical_frame_id>
-                <camera_info_topic>camera/depth/camera_info</camera_info_topic>
-                <horizontal_fov>1.05</horizontal_fov>
-                <pose>0 0 0 0 0 0</pose>
-                <image>
-                    <width>640</width>
-                    <height>480</height>
-                    <format>R_FLOAT32</format>
-                </image>
-                <clip>
-                    <near>0.1</near>
-                    <far>10.0</far>
-                </clip>
-            </camera>
-        </sensor>
-    </gazebo>
-    <link name="camera_depth_optical_frame" />
-    <joint name="camera_depth_optical_frame_joint" type="fixed">
-        <parent link="camera_link" />
-        <child link="camera_depth_optical_frame" />
-        <origin xyz="0 0 0" rpy="-1.57079632679 0 -1.57079632679" />
-    </joint>
-    <joint name="camera_joint" type="fixed">
-        <parent link="base_link" />
-        <child link="camera_link" />
-        <origin xyz="0.2 0 0.0" rpy="0 0 0" />
+        <child link="camera_rgbd_optical_frame" />
+        <origin xyz="0 0 0" rpy="0 0 0" />
     </joint>
     <!-- ===================== -->
@@ -112,4 +78,5 @@
         </collision>
     </link>
+    <!-- TODO this imu topic is not working -->
     <gazebo reference="imu_link">
         <sensor name="imu_sensor" type="imu">
@@ -117,5 +84,8 @@
             <update_rate>1</update_rate>
             <visualize>true</visualize>
-            <topic>imu</topic>
+            <topic>/${robot_namespace}/imu</topic>
+            <plugin filename="gz-sim-imu-system"
+                name="gz::sim::systems::Imu">
+            </plugin>
         </sensor>
     </gazebo>
