Commit message: working control simulation

File: src/drone_description/description/components/rotor.xacro (robot description, xacro)
@@ -39,5 +39,6 @@
                 <rotorDragCoefficient>8.06428e-05</rotorDragCoefficient>
                 <rollingMomentCoefficient>1e-06</rollingMomentCoefficient>
-                <rotorVelocitySlowdownSim>10</rotorVelocitySlowdownSim>
+                <!-- set to 1 for direct rotor velocity simulation (less artificial slowdown) -->
+                <rotorVelocitySlowdownSim>1</rotorVelocitySlowdownSim>
                 <motorType>velocity</motorType>
             </plugin>

File: src/drone_description/description/drone.urdf.xacro (robot description, xacro)
@@ -26,8 +26,8 @@
         </xacro:inertial_box>
     </link>
-    <xacro:rotor suffix="0" x="0.15" y="0.15" ccw="1" />  <!-- Front Left -->
-    <xacro:rotor suffix="1" x="-0.15" y="-0.15" ccw="1" />  <!-- Rear Right -->
-    <xacro:rotor suffix="2" x="0.15" y="-0.15" ccw="-1" /> <!-- Front Right -->
-    <xacro:rotor suffix="3" x="-0.15" y="0.15" ccw="-1" /> <!-- Rear Left -->
+    <xacro:rotor suffix="0" x="0.15" y="0.15" ccw="-1" />  <!-- Front Left -->
+    <xacro:rotor suffix="1" x="-0.15" y="-0.15" ccw="-1" />  <!-- Rear Right -->
+    <xacro:rotor suffix="2" x="0.15" y="-0.15" ccw="1" /> <!-- Front Right -->
+    <xacro:rotor suffix="3" x="-0.15" y="0.15" ccw="1" /> <!-- Rear Left -->
     <xacro:include filename="sensors.xacro" />
     <gazebo>

File: src/drone_description/description/sensors.xacro (robot description, xacro)
@@ -6,5 +6,5 @@
     <link name="camera_link">
         <inertial>
-            <mass value="0.05" />
+            <mass value="0.0" />
             <inertia ixx="0.0001" ixy="0.0" ixz="0.0" iyy="0.0001" iyz="0.0" izz="0.0001" />
         </inertial>
@@ -61,5 +61,5 @@
     <link name="imu_link">
         <inertial>
-            <mass value="0.05" />
+            <mass value="0.0" />
             <inertia ixx="0.0001" ixy="0.0" ixz="0.0" iyy="0.0001" iyz="0.0" izz="0.0001" />
         </inertial>
